Commit message: update

File: urdf/ur_sim.urdf.xacro (robot description, xacro)
@@ -5,4 +5,5 @@
    <!-- import main macro -->
    <xacro:include filename="$(find ur_description)/urdf/ur_macro.xacro"/>
+   <xacro:include filename="$(find ur_description)/urdf/ur5_hammer_eef.urdf.xacro"/>
    <!-- possible 'ur_type' values: ur3, ur3e, ur5, ur5e, ur10, ur10e, ur16e, ur20, ur30 -->
    <!-- the default value should raise an error in case this was called without defining the type -->
@@ -92,6 +93,8 @@
      trajectory_port="$(arg trajectory_port)"
      >
-     <origin xyz="0 0 0.3" rpy="0 0 0" />          <!-- position robot in the world -->
+     <origin xyz="0 0 0" rpy="0 0 0" />          <!-- position robot in the world -->
    </xacro:ur_robot>
+  <!-- hammer eef -->
+  <xacro:hammer_eef prefix="" />
    <xacro:if value="$(arg sim_gazebo)">
     <!-- Gazebo plugins -->
