Commit message: update initial positions and rviz configuration for improved robot control

File: urdf/ur_hammer.urdf.xacro (robot description, xacro)
@@ -90,5 +90,5 @@
      trajectory_port="$(arg trajectory_port)"
      >
-     <origin xyz="0 0 0" rpy="0 0 0" />          <!-- position robot in the world -->
+     <origin xyz="0 0 0" rpy="0 0 3.92699" />          <!-- position robot in the world -->
    </xacro:ur_robot>
   <!-- hammer eef -->

File: urdf/ur_sim.urdf.xacro (robot description, xacro)
@@ -93,5 +93,5 @@
      trajectory_port="$(arg trajectory_port)"
      >
-     <origin xyz="0 0 0" rpy="0 0 0" />          <!-- position robot in the world -->
+     <origin xyz="0 0 0" rpy="0 0 3.92699" />     <!-- position robot in the world -->
    </xacro:ur_robot>
   <!-- hammer eef -->
